File: Projekti/Single_transitor_AMP/Single_transistor_AMP.sch (KiCad schematic (older format))
At the start: 10 parts, among them P1 CONN_01X02, P2 CONN_01X02, Q1 BC549

Commit message: Pabeigts 3rd majasdarbs
Parts:
- removed C3: C_Variable, symbol C_Variable
- added C3: 2.2uF, Capacitors_THT:CP_Radial_D10.0mm_P2.50mm, symbol C
- C1: value C -> 2.2uF; footprint (none) -> Capacitors_THT:CP_Radial_D10.0mm_P2.50mm
- C2: value C -> 22uF; footprint (none) -> Capacitors_THT:CP_Radial_D10.0mm_P2.50mm
- P1, P2: value CONN_01X02 -> CONN; footprint (none) -> Connectors:AK300-2
- R1: value R -> 22K; footprint Resistors_THT:R_Axial_DIN0309_L9.0mm_D3.2mm_P15.24mm_Horizontal -> Resistors_THT:R_Axial_DIN0414_L11.9mm_D4.5mm_P25.40mm_Horizontal
- R2: value R -> 6.8K
- R3: value R -> 4.7K
- R4: value R -> 1.8K
Connections:
- net at Q1.1 (C), R3.1: now also C3.2
- net at P2.1 (P1): now also C3.1
Other:
- moved on the sheet: C1, C2, P1, Q1, R1, R2, R3, R4
