File: Projekti/Single_transitor_AMP/Single_transistor_AMP.sch (KiCad schematic (older format))
At the start: 10 parts, among them P1 CONN, P2 CONN, Q1 BC549

Commit message: pebeigts md par layout
Parts:
- added P3: CONN, Connectors:AK300-2, symbol CONN_01X02
Connections:
- net +24V: now also P3.1 (P1)
- net GND: now also P3.2 (P2)
Changed lines of the file:
@@
 $EndComp
 Wire Wire Line
-	5050 3300 5250 3300
-Wire Wire Line
-	5250 3300 5500 3300
-Wire Wire Line
-	5250 3000 5250 3300
-Wire Wire Line
-	5250 3300 5250 3650
+	5050 3300 5500 3300
+Wire Wire Line
+	5250 3000 5250 3650
 Connection ~ 5250 3300
 $Comp
@@
 $EndComp
 Wire Wire Line
-	5800 3500 5800 3600
-Wire Wire Line
-	5800 3600 5800 3650
+	5800 3500 5800 3650
 Wire Wire Line
 	5250 3950 5250 4150
 Wire Wire Line
-	5250 4150 5800 4150
-Wire Wire Line
-	5800 4150 6350 4150
-Wire Wire Line
-	5800 3950 5800 4150
-Wire Wire Line
-	5800 4150 5800 4300
+	5250 4150 6350 4150
+Wire Wire Line
+	5800 3950 5800 4300
 $Comp
 L C C2
@@
 Connection ~ 5800 3600
 Wire Wire Line
-	6350 3950 6350 4150
-Wire Wire Line
-	6350 4150 6350 4250
+	6350 3950 6350 4250
 Connection ~ 5800 4150
 Wire Wire Line
-	5250 2650 5800 2650
-Wire Wire Line
-	5800 2650 6150 2650
-Wire Wire Line
-	6150 2650 6450 2650
+	5250 2650 6450 2650
 Wire Wire Line
 	5250 2650 5250 2700
@@
 	5800 2650 5800 2700
 Wire Wire Line
-	5800 3000 5800 3050
-Wire Wire Line
-	5800 3050 5800 3100
+	5800 3000 5800 3100
 Wire Wire Line
 	5800 3050 6400 3050
@@
 	0    1    1    0
 $EndComp
+$Comp
+L CONN_01X02 P3
+U 1 1 59143DD1
+P 7350 4150
+F 0 "P3" H 7350 4300 50  0000 C CNN
+F 1 "CONN" V 7450 4150 50  0000 C CNN
+F 2 "Connectors:AK300-2" H 7350 4150 50  0001 C CNN
+F 3 "" H 7350 4150 50  0000 C CNN
+	1    7350 4150
+	1    0    0    -1
+$EndComp
+Wire Wire Line
+	7150 4200 7050 4200
+Wire Wire Line
+	7050 4200 7050 4350
+$Comp
+L GND #PWR07
+U 1 1 59143E4A
+P 7050 4350
+F 0 "#PWR07" H 7050 4100 50  0001 C CNN
+F 1 "GND" H 7050 4200 50  0000 C CNN
+F 2 "Connectors:1pin" H 7050 4350 50  0001 C CNN
+F 3 "" H 7050 4350 50  0000 C CNN
+	1    7050 4350
+	1    0    0    -1
+$EndComp
+Wire Wire Line
+	7150 4100 7050 4100
+Wire Wire Line
+	7050 4100 7050 4000
+$Comp
+L +24V #PWR08
+U 1 1 59143EA3
+P 7050 4000
+F 0 "#PWR08" H 7050 3850 50  0001 C CNN
+F 1 "+24V" H 7050 4140 50  0000 C CNN
+F 2 "Connectors:1pin" H 7050 4000 50  0001 C CNN
+F 3 "" H 7050 4000 50  0000 C CNN
+	1    7050 4000
+	1    0    0    -1
+$EndComp
 $EndSCHEMATC

Commit message: tika izstradata traseshana un izvedoti gerber faili
Parts:
- R1: footprint Resistors_THT:R_Axial_DIN0414_L11.9mm_D4.5mm_P25.40mm_Horizontal -> Resistors_THT:R_Axial_DIN0309_L9.0mm_D3.2mm_P15.24mm_Horizontal
Changed lines of the file:
@@
 F 0 "R1" V 5330 2850 50  0000 C CNN
 F 1 "22K" V 5250 2850 50  0000 C CNN
-F 2 "Resistors_THT:R_Axial_DIN0414_L11.9mm_D4.5mm_P25.40mm_Horizontal" V 5180 2850 50  0001 C CNN
+F 2 "Resistors_THT:R_Axial_DIN0309_L9.0mm_D3.2mm_P15.24mm_Horizontal" V 5180 2850 50  0001 C CNN
 F 3 "https://www.digchip.com/datasheets/parts/datasheet/1838/CFR-50JB-22K-pdf.php" H 5250 2850 50  0001 C CNN
 	1    5250 2850
