File: Projekti/Single_transitor_AMP/Single_transistor_AMP.kicad_pcb (KiCad board)
At the start: 2 copper layers, 76.2 x 63.5 mm, 11 parts, among them P1 CONN, P2 CONN, P3 CONN, Q1 BC549

Commit message: izmainas
Parts:
- added G***: LOGO, logo:LOGO, F.Cu at (135.6, 120.4)
Changed lines of the file:
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@@
 (kicad_pcb (version 4) (host pcbnew 4.0.5)
   (general
-    (links 16)
+    (links 0)
     (no_connects 0)
     (area 120.574999 69.774999 196.925001 133.425001)
@@
     (tracks 31)
     (zones 0)
-    (modules 11)
+    (modules 12)
     (nets 8)
   )
@@
     )
   )
+  (module logo:LOGO (layer F.Cu)
+    (at 135.636 120.396)
+    (fp_text reference G*** (at 0 0) (layer F.SilkS) hide
+      (effects (font (thickness 0.3)))
+    )
+    (fp_text value LOGO (at 0.75 0) (layer F.SilkS) hide
+      (effects (font (thickness 0.3)))
+    )
+    (fp_poly (pts (xy -3.415894 -1.911552) (xy -3.38419 -1.804533) (xy -3.317609 -1.553375) (xy -3.230205 -1.211162)
+      (xy -3.225051 -1.190665) (xy -3.086466 -0.703785) (xy -2.910904 -0.171872) (xy -2.786746 0.161176)
+      (xy -2.637534 0.57587) (xy -2.5154 0.989706) (xy -2.454571 1.270029) (xy -2.3876 1.715976)
+      (xy -1.8796 1.388372) (xy -1.599194 1.187939) (xy -1.398112 1.007542) (xy -1.331148 0.911383)
+      (xy -1.300142 0.673436) (xy -1.302052 0.37302) (xy -1.330828 0.082113) (xy -1.380422 -0.127309)
+      (xy -1.423429 -0.18661) (xy -1.540724 -0.294395) (xy -1.672825 -0.501087) (xy -1.755376 -0.689629)
+      (xy -1.723608 -0.802448) (xy -1.545916 -0.909714) (xy -1.472946 -0.944861) (xy -1.244912 -1.042265)
+      (xy -1.101402 -1.034481) (xy -0.953936 -0.900389) (xy -0.869029 -0.800723) (xy -0.68184 -0.535562)
+      (xy -0.558838 -0.284461) (xy -0.549065 -0.251385) (xy -0.525135 -0.005894) (xy -0.529982 0.366407)
+      (xy -0.559976 0.791727) (xy -0.611491 1.196276) (xy -0.623671 1.266107) (xy -0.584676 1.446529)
+      (xy -0.4572 1.50657) (xy -0.112061 1.669907) (xy 0.209435 1.986457) (xy 0.475147 2.40641)
+      (xy 0.652928 2.879957) (xy 0.7112 3.317118) (xy 0.695406 3.484137) (xy 0.609376 3.541891)
+      (xy 0.395132 3.519341) (xy 0.3302 3.507445) (xy 0.084572 3.458059) (xy -0.04982 3.424254)
+      (xy -0.057878 3.419938) (xy -0.087418 3.322068) (xy -0.153563 3.094585) (xy -0.187597 2.976338)
+      (xy -0.34193 2.569647) (xy -0.535076 2.341268) (xy -0.796311 2.266536) (xy -1.006232 2.286717)
+      (xy -1.282365 2.357968) (xy -1.475702 2.442183) (xy -1.489555 2.452425) (xy -1.629118 2.48758)
+      (xy -1.673351 2.443333) (xy -1.832479 2.345624) (xy -2.071346 2.431029) (xy -2.202284 2.528179)
+      (xy -2.319689 2.637779) (xy -2.371011 2.751853) (xy -2.360775 2.92899) (xy -2.293508 3.227777)
+      (xy -2.265089 3.341137) (xy -2.190806 3.673137) (xy -2.153121 3.919574) (xy -2.158417 4.021083)
+      (xy -2.284511 4.070565) (xy -2.524981 4.123573) (xy -2.561238 4.129683) (xy -2.912453 4.186678)
+      (xy -3.085409 3.386189) (xy -3.169322 2.904077) (xy -3.224611 2.402115) (xy -3.239601 1.987061)
+      (xy -3.239356 1.97865) (xy -3.244928 1.67923) (xy -3.287616 1.362067) (xy -3.377674 0.982305)
+      (xy -3.525358 0.495089) (xy -3.692974 -0.005357) (xy -3.904555 -0.62964) (xy -4.049194 -1.089624)
+      (xy -4.128431 -1.412323) (xy -4.143808 -1.624752) (xy -4.096864 -1.753922) (xy -3.989142 -1.826847)
+      (xy -3.822182 -1.870542) (xy -3.799619 -1.874845) (xy -3.55702 -1.911799) (xy -3.423312 -1.915743)
+      (xy -3.415894 -1.911552)) (layer F.SilkS) (width 0.01))
+    (fp_poly (pts (xy 1.364104 -2.09921) (xy 1.575007 -2.031922) (xy 1.765944 -1.915896) (xy 1.786404 -1.754945)
+      (xy 1.781192 -1.737258) (xy 1.795811 -1.584578) (xy 1.870875 -1.291352) (xy 1.989799 -0.905068)
+      (xy 2.135999 -0.473215) (xy 2.292891 -0.04328) (xy 2.44389 0.337249) (xy 2.572411 0.620883)
+      (xy 2.648855 0.747231) (xy 2.777837 0.756064) (xy 3.019769 0.672513) (xy 3.324331 0.525154)
+      (xy 3.641201 0.34257) (xy 3.920058 0.153337) (xy 4.11058 -0.013963) (xy 4.1656 -0.114185)
+      (xy 4.204587 -0.23988) (xy 4.355575 -0.295155) (xy 4.572 -0.3048) (xy 4.833476 -0.291353)
+      (xy 4.949713 -0.22616) (xy 4.978154 -0.071945) (xy 4.9784 -0.041085) (xy 4.888853 0.308271)
+      (xy 4.654765 0.640517) (xy 4.327968 0.886307) (xy 4.262963 0.916154) (xy 3.948654 1.046345)
+      (xy 4.539727 1.362579) (xy 5.215449 1.741748) (xy 5.722509 2.074454) (xy 6.082697 2.385071)
+      (xy 6.317805 2.697973) (xy 6.449622 3.037537) (xy 6.499939 3.428138) (xy 6.5024 3.558056)
+      (xy 6.5024 3.9624) (xy 6.085129 3.9624) (xy 5.815929 3.94459) (xy 5.715382 3.882891)
+      (xy 5.721758 3.821943) (xy 5.732715 3.638434) (xy 5.69238 3.35926) (xy 5.675022 3.285016)
+      (xy 5.570031 3.010065) (xy 5.383581 2.798914) (xy 5.098593 2.607162) (xy 4.753773 2.400938)
+      (xy 4.421996 2.198901) (xy 4.296783 2.121179) (xy 4.003294 1.991909) (xy 3.618741 1.890504)
+      (xy 3.407474 1.858444) (xy 2.844181 1.800307) (xy 2.906144 2.144753) (xy 2.972618 2.455776)
+      (xy 3.067697 2.83684) (xy 3.109308 2.989078) (xy 3.184923 3.276851) (xy 3.224709 3.469122)
+      (xy 3.225454 3.513417) (xy 3.119437 3.546035) (xy 2.888852 3.59579) (xy 2.826026 3.607802)
+      (xy 2.582844 3.641234) (xy 2.45732 3.588903) (xy 2.379889 3.404087) (xy 2.347879 3.286664)
+      (xy 2.281067 3.020897) (xy 2.222975 2.74862) (xy 2.161372 2.406644) (xy 2.084027 1.931779)
+      (xy 2.076803 1.88622) (xy 2.011174 1.600005) (xy 1.894105 1.200645) (xy 1.748279 0.764195)
+      (xy 1.713224 0.66702) (xy 1.536851 0.185629) (xy 1.352026 -0.318963) (xy 1.196037 -0.744953)
+      (xy 1.183211 -0.779989) (xy 1.058543 -1.207345) (xy 1.000915 -1.597482) (xy 1.010651 -1.90801)
+      (xy 1.088073 -2.096541) (xy 1.172901 -2.133601) (xy 1.364104 -2.09921)) (layer F.SilkS) (width 0.01))
+  )
   (gr_line (start 133.35 133.35) (end 184.15 133.35) (layer Edge.Cuts) (width 0.15))
