File: Projekti/Battery/battery.sch (KiCad schematic (older format))
At the start: 4 parts

Commit message: pabeigts md ar bateriju turetajiem
Parts:
- removed BT1: Battery_Cell, Battery_Holders:SMTU2032, symbol Battery_Cell
- removed R1: R, symbol R
- BT2: footprint Battery_Holders:S8211R -> Battery_Holders:CH28-2032LF
Other:
- moved on the sheet: R2
Changed lines of the file:
@@
 LIBS:contrib
 LIBS:valves
+LIBS:battery-cache
 EELAYER 25 0
 EELAYER END
@@
 encoding utf-8
 Sheet 1 1
-Title ""
-Date ""
-Rev ""
-Comp ""
+Title "Battery"
+Date "10.04.2017"
+Rev "1.0"
+Comp "VeA"
 Comment1 ""
 Comment2 ""
@@
 $EndDescr
 $Comp
-L Battery_Cell BT1
-U 1 1 58DCBB7E
-P 1800 3250
-F 0 "BT1" H 1900 3350 50  0000 L CNN
-F 1 "Battery_Cell" H 1900 3250 50  0000 L CNN
-F 2 "Battery_Holders:SMTU2032" V 1800 3310 50  0001 C CNN
-F 3 "" V 1800 3310 50  0000 C CNN
-	1    1800 3250
+L R R2
+U 1 1 58DCBF78
+P 6200 3950
+F 0 "R2" V 6280 3950 50  0000 C CNN
+F 1 "R" V 6200 3950 50  0000 C CNN
+F 2 "" V 6130 3950 50  0000 C CNN
+F 3 "" H 6200 3950 50  0000 C CNN
+	1    6200 3950
+	0    1    1    0
+$EndComp
+Wire Wire Line
+	5850 4100 5850 3950
+Wire Wire Line
+	5850 3950 6050 3950
+Wire Wire Line
+	6350 3950 6550 3950
+Wire Wire Line
+	6550 3950 6550 4550
+Wire Wire Line
+	6550 4550 5850 4550
+Wire Wire Line
+	5850 4550 5850 4400
+$Comp
+L Battery_Cell BT2
+U 1 1 58F66F0C
+P 5850 4300
+F 0 "BT2" H 5950 4400 50  0000 L CNN
+F 1 "Battery_Cell" H 5950 4300 50  0000 L CNN
+F 2 "Battery_Holders:CH28-2032LF" V 5850 4360 50  0001 C CNN
+F 3 "" V 5850 4360 50  0000 C CNN
+	1    5850 4300
 	1    0    0    -1
 $EndComp
-$Comp
-L R R1
-U 1 1 58DCBBE7
-P 2800 3200
-F 0 "R1" V 2880 3200 50  0000 C CNN
-F 1 "R" V 2800 3200 50  0000 C CNN
-F 2 "" V 2730 3200 50  0000 C CNN
-F 3 "" H 2800 3200 50  0000 C CNN
-	1    2800 3200
-	1    0    0    -1
-$EndComp
-Wire Wire Line
-	1800 3050 1800 2950
-Wire Wire Line
-	1800 2950 2800 2950
-Wire Wire Line
-	2800 2950 2800 3050
-Wire Wire Line
-	2800 3350 2800 3550
-Wire Wire Line
-	2800 3550 1800 3550
-Wire Wire Line
-	1800 3550 1800 3350
-$Comp
-L R R2
-U 1 1 58DCBF78
-P 4150 2900
-F 0 "R2" V 4230 2900 50  0000 C CNN
-F 1 "R" V 4150 2900 50  0000 C CNN
-F 2 "" V 4080 2900 50  0000 C CNN
-F 3 "" H 4150 2900 50  0000 C CNN
-	1    4150 2900
-	0    1    1    0
-$EndComp
-$Comp
-L Battery_Cell BT2
-U 1 1 58DCBFC5
-P 3800 3250
-F 0 "BT2" H 3900 3350 50  0000 L CNN
-F 1 "Battery_Cell" H 3900 3250 50  0000 L CNN
-F 2 "Battery_Holders:S8211R" V 3800 3310 50  0001 C CNN
-F 3 "" V 3800 3310 50  0000 C CNN
-	1    3800 3250
-	1    0    0    -1
-$EndComp
-Wire Wire Line
-	3800 3050 3800 2900
-Wire Wire Line
-	3800 2900 4000 2900
-Wire Wire Line
-	4300 2900 4500 2900
-Wire Wire Line
-	4500 2900 4500 3500
-Wire Wire Line
-	4500 3500 3800 3500
-Wire Wire Line
-	3800 3500 3800 3350
 $EndSCHEMATC
