File: Projekti/18W_AMP/18W_AMP.kicad_pcb (KiCad board)
At the start: 2 copper layers, 116.3 x 110.7 mm, 24 parts, among them P1 INPUT, P2 OUTPUT, P3 CONN_01X02, Q1 BD908, Q2 BD907, U1 TDA2030A

Commit message: principā pabeigts kursa darbs, vēl daži sīkumi
Parts:
- moved D2 1.02 mm to (154.4, 51.3)
Routing:
- net GND: track 328.5 -> 327.5 mm
- net Net-(C8-Pad1): track 224.1 -> 223.5 mm
- added copper zone on B.Cu, net GND
- added copper zone on F.Cu, net GND
Other:
- outline, holes or cut-outs redrawn

Commit message: Pabeigts kursa darbs
Parts:
- added G***: LOGO, logo:LOGO, F.Cu at (74.2, 52.8)
Changed lines of the file:
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@@
 (kicad_pcb (version 4) (host pcbnew 4.0.5)
   (general
-    (links 41)
+    (links 0)
     (no_connects 0)
     (area 59.868999 26.409198 177.292001 137.743001)
@@
     (tracks 225)
     (zones 0)
-    (modules 24)
+    (modules 25)
     (nets 13)
   )
@@
       (drillshape 0)
       (scaleselection 1)
-      (outputdirectory Gerber/))
+      (outputdirectory svg_faili/))
   )
   (net 0 "")
@@
     )
   )
+  (module logo:LOGO (layer F.Cu)
+    (at 74.168 52.832)
+    (fp_text reference G*** (at 0 0) (layer F.SilkS) hide
+      (effects (font (thickness 0.3)))
+    )
+    (fp_text value LOGO (at 0.75 0) (layer F.SilkS) hide
+      (effects (font (thickness 0.3)))
+    )
+    (fp_poly (pts (xy -3.789967 -2.139775) (xy -3.703821 -1.87624) (xy -3.610815 -1.478709) (xy -3.517472 -0.981297)
+      (xy -3.430313 -0.418117) (xy -3.35586 0.176717) (xy -3.309173 0.6604) (xy -3.192358 2.0828)
+      (xy -2.717047 1.35886) (xy -2.346484 0.708965) (xy -2.132234 0.100969) (xy -2.057138 -0.529047)
+      (xy -2.078416 -1.019901) (xy -2.106333 -1.386746) (xy -2.094516 -1.61538) (xy -2.030162 -1.768998)
+      (xy -1.900466 -1.910795) (xy -1.897307 -1.913766) (xy -1.652947 -2.143331) (xy -1.588474 -1.820966)
+      (xy -1.529542 -1.105625) (xy -1.610148 -0.34268) (xy -1.815133 0.399579) (xy -2.129333 1.052861)
+      (xy -2.27289 1.261841) (xy -2.461445 1.521701) (xy -2.524849 1.661874) (xy -2.468644 1.71827)
+      (xy -2.344718 1.7272) (xy -2.13893 1.814482) (xy -1.884045 2.048688) (xy -1.60713 2.388357)
+      (xy -1.335253 2.792026) (xy -1.095482 3.218233) (xy -0.914884 3.625517) (xy -0.820526 3.972415)
+      (xy -0.812881 4.073653) (xy -0.882711 4.342587) (xy -0.998601 4.505453) (xy -1.201757 4.653915)
+      (xy -1.303652 4.633996) (xy -1.3208 4.53485) (xy -1.378199 4.304718) (xy -1.530534 3.965239)
+      (xy -1.748015 3.567484) (xy -2.000852 3.162521) (xy -2.259255 2.801421) (xy -2.479225 2.548967)
+      (xy -2.786957 2.284452) (xy -3.005957 2.197368) (xy -3.154691 2.294536) (xy -3.251629 2.582776)
+      (xy -3.292502 2.849357) (xy -3.344387 3.282103) (xy -3.399239 3.738958) (xy -3.412794 3.851726)
+      (xy -3.516305 4.282738) (xy -3.71833 4.579909) (xy -3.727221 4.588326) (xy -3.981655 4.826)
+      (xy -3.911407 4.1656) (xy -3.887132 3.83124) (xy -3.866766 3.347242) (xy -3.851872 2.767157)
+      (xy -3.844013 2.144532) (xy -3.843216 1.8288) (xy -3.847667 1.163391) (xy -3.862491 0.650319)
+      (xy -3.892684 0.23879) (xy -3.943243 -0.121988) (xy -4.019164 -0.482808) (xy -4.102872 -0.810685)
+      (xy -4.360472 -1.773769) (xy -4.143726 -2.004485) (xy -3.97326 -2.166207) (xy -3.863786 -2.235171)
+      (xy -3.862733 -2.235201) (xy -3.789967 -2.139775)) (layer F.SilkS) (width 0.01))
+    (fp_poly (pts (xy 1.391633 -2.139775) (xy 1.477779 -1.87624) (xy 1.570785 -1.478709) (xy 1.664128 -0.981297)
+      (xy 1.751287 -0.418117) (xy 1.82574 0.176717) (xy 1.872427 0.6604) (xy 1.989242 2.0828)
+      (xy 2.464553 1.35886) (xy 2.835116 0.708965) (xy 3.049366 0.100969) (xy 3.124462 -0.529047)
+      (xy 3.103184 -1.019901) (xy 3.075267 -1.386746) (xy 3.087084 -1.61538) (xy 3.151438 -1.768998)
+      (xy 3.281134 -1.910795) (xy 3.284293 -1.913766) (xy 3.528653 -2.143331) (xy 3.593126 -1.820966)
+      (xy 3.652058 -1.105625) (xy 3.571452 -0.34268) (xy 3.366467 0.399579) (xy 3.052267 1.052861)
+      (xy 2.90871 1.261841) (xy 2.720155 1.521701) (xy 2.656751 1.661874) (xy 2.712956 1.71827)
+      (xy 2.836882 1.7272) (xy 3.04267 1.814482) (xy 3.297555 2.048688) (xy 3.57447 2.388357)
+      (xy 3.846347 2.792026) (xy 4.086118 3.218233) (xy 4.266716 3.625517) (xy 4.361074 3.972415)
+      (xy 4.368719 4.073653) (xy 4.298889 4.342587) (xy 4.182999 4.505453) (xy 3.979843 4.653915)
+      (xy 3.877948 4.633996) (xy 3.8608 4.53485) (xy 3.803401 4.304718) (xy 3.651066 3.965239)
+      (xy 3.433585 3.567484) (xy 3.180748 3.162521) (xy 2.922345 2.801421) (xy 2.702375 2.548967)
+      (xy 2.394643 2.284452) (xy 2.175643 2.197368) (xy 2.026909 2.294536) (xy 1.929971 2.582776)
+      (xy 1.889098 2.849357) (xy 1.837213 3.282103) (xy 1.782361 3.738958) (xy 1.768806 3.851726)
+      (xy 1.665295 4.282738) (xy 1.46327 4.579909) (xy 1.454379 4.588326) (xy 1.199945 4.826)
+      (xy 1.270193 4.1656) (xy 1.294468 3.83124) (xy 1.314834 3.347242) (xy 1.329728 2.767157)
+      (xy 1.337587 2.144532) (xy 1.338384 1.8288) (xy 1.333933 1.163391) (xy 1.319109 0.650319)
+      (xy 1.288916 0.23879) (xy 1.238357 -0.121988) (xy 1.162436 -0.482808) (xy 1.078728 -0.810685)
+      (xy 0.821128 -1.773769) (xy 1.037874 -2.004485) (xy 1.20834 -2.166207) (xy 1.317814 -2.235171)
+      (xy 1.318867 -2.235201) (xy 1.391633 -2.139775)) (layer F.SilkS) (width 0.01))
+    (fp_poly (pts (xy 0.217725 4.250351) (xy 0.289449 4.410064) (xy 0.285742 4.443526) (xy 0.180885 4.605594)
+      (xy 0.008712 4.652748) (xy -0.141012 4.569426) (xy -0.166198 4.521879) (xy -0.167369 4.323348)
+      (xy -0.12192 4.24688) (xy 0.051001 4.181678) (xy 0.217725 4.250351)) (layer F.SilkS) (width 0.01))
+    (fp_poly (pts (xy 5.196125 4.250351) (xy 5.267849 4.410064) (xy 5.264142 4.443526) (xy 5.159285 4.605594)
+      (xy 4.987112 4.652748) (xy 4.837388 4.569426) (xy 4.812202 4.521879) (xy 4.811031 4.323348)
+      (xy 4.85648 4.24688) (xy 5.029401 4.181678) (xy 5.196125 4.250351)) (layer F.SilkS) (width 0.01))
+  )
   (gr_arc (start 76.708 43.688) (end 59.944 43.688) (angle 90) (layer Edge.Cuts) (width 0.15))
