File: Projekti/PWR_Supply/12Vreg.sch (KiCad schematic (older format))
At the start: 3 parts, among them U2 LM7812

Commit message: izmainas
Connections:
- net VCC renamed +12V
Changed lines of the file:
@@
 $EndComp
 $Comp
-L GND #PWR03
+L GND #PWR06
 U 1 1 58D11FC4
 P 5600 4050
-F 0 "#PWR03" H 5600 3800 50  0001 C CNN
+F 0 "#PWR06" H 5600 3800 50  0001 C CNN
 F 1 "GND" H 5600 3900 50  0000 C CNN
 F 2 "" H 5600 4050 50  0000 C CNN
@@
 GND
 Text HLabel 4400 3450 0    60   Input ~ 0
-VCC
++12V
 Connection ~ 4750 3450
 $EndSCHEMATC
