File: Projekti/PWR_Supply/220V_AC.sch (KiCad schematic (older format))
At the start: 4 parts, among them P1 CONN_01X02, T1 Transformer_1P_1S

Commit message: pabeigts md ar bateriju turetajiem
Connections:
- net VCC renamed +12V
Changed lines of the file:
@@
 	6050 3800 6050 3600
 Text HLabel 6500 3100 2    60   Input ~ 0
-VCC
++12V
 Text HLabel 6550 3800 2    60   Input ~ 0
 GND

Commit message: izmainas
Changed lines of the file:
@@
 Wire Wire Line
 	6050 3800 6050 3600
-Text HLabel 6500 3100 2    60   Input ~ 0
+Text HLabel 6500 3100 2    60   Output ~ 0
 +12V
-Text HLabel 6550 3800 2    60   Input ~ 0
+Text HLabel 6550 3800 2    60   Output ~ 0
 GND
 Connection ~ 6050 3100
