File: Projekti/PWR_Supply/3_3Vreg.sch (KiCad schematic (older format))
At the start: 3 parts, among them U3 LM3940

Commit message: izmainas
Parts:
- C6: value 0.47uF -> 10uF
- C7: value 33uF -> 10uF
- U3: value LM3940 -> LT1086-3.3
Connections:
- net VCC renamed +12V
Changed lines of the file:
@@
 AR Path="/58D1154E/58D15683" Ref="U3"  Part="1"
 F 0 "U3" H 6300 5250 60  0000 C CNN
-F 1 "LM3940" H 6700 5250 60  0000 C CNN
+F 1 "LT1086-3.3" H 6700 5250 60  0000 C CNN
 F 2 "" H 8050 4300 60  0001 C CNN
 F 3 "" H 8050 4300 60  0001 C CNN
@@
 P 5600 3800
 F 0 "C6" H 5625 3900 50  0000 L CNN
-F 1 "0.47uF" H 5625 3700 50  0000 L CNN
+F 1 "10uF" H 5625 3700 50  0000 L CNN
 F 2 "" H 5600 3800 50  0000 C CNN
 F 3 "" H 5600 3800 50  0000 C CNN
@@
 P 7550 3800
 F 0 "C7" H 7575 3900 50  0000 L CNN
-F 1 "33uF" H 7575 3700 50  0000 L CNN
+F 1 "10uF" H 7575 3700 50  0000 L CNN
 F 2 "" H 7550 3800 50  0000 C CNN
 F 3 "" H 7550 3800 50  0000 C CNN
@@
 	7550 3550 7550 3650
 $Comp
-L GND #PWR04
+L GND #PWR07
 U 1 1 58D1585E
 P 6600 4250
-F 0 "#PWR04" H 6600 4000 50  0001 C CNN
+F 0 "#PWR07" H 6600 4000 50  0001 C CNN
 F 1 "GND" H 6600 4100 50  0000 C CNN
 F 2 "" H 6600 4250 50  0000 C CNN
@@
 Connection ~ 7550 3550
 Text HLabel 5250 3550 0    60   Input ~ 0
-VCC
++12V
 Connection ~ 5600 3550
 Text HLabel 7900 4150 2    60   Input ~ 0
