File: Projekti/PWR_Supply/5Vreg.sch (KiCad schematic (older format))
At the start: 3 parts, among them U1 7805

Commit message: izmainas
Connections:
- net VCC renamed +12V
Changed lines of the file:
@@
 $EndComp
 $Comp
-L GND #PWR01
+L GND #PWR03
 U 1 1 58D129DD
 P 5500 3400
-F 0 "#PWR01" H 5500 3150 50  0001 C CNN
+F 0 "#PWR03" H 5500 3150 50  0001 C CNN
 F 1 "GND" H 5500 3250 50  0000 C CNN
 F 2 "" H 5500 3400 50  0000 C CNN
@@
 Connection ~ 6350 2750
 Text HLabel 4400 2750 0    60   Input ~ 0
-VCC
++12V
 Connection ~ 4650 2750
 $EndSCHEMATC
